Commit message: 记录

File: generated/urdf/总装/mujoco.urdf (robot description, URDF)
Before this commit: robot 总装, 13 links, 12 joints
Links:
- link base_link: geometry collision mesh filename=/home/coffee/rm_sim_spear/assets/总装_urdf/meshes/Board_31iW_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; collision mesh filename=/home/coffee/rm_sim_spear/assets/总装_urdf/meshes/CONN_TH_XT3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
- link link_6: geometry collision mesh filename=/home/coffee/rm_sim_spear/assets/总装_urdf/meshes/RAU6005交叉滚子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; collision mesh filename=/home/coffee/rm_sim_spear/assets/总装_urdf/meshes/TPU上壳_默认_37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
Joints:
- joint link_1_joint: axis 1.1102230246251568E-16 -1.3877787807814459E-16 1 -> 1.1102230246251568E-16 -2.2204460492503136E-16 1
- joint link_3_joint: axis 2.2204460492503131E-16 -8.3266726846886741E-17 1 -> 2.7755575615628914E-16 -1.6653345369377348E-16 1
- joint link_4_joint: axis -8.3266726846886765E-17 -5.5511151231257839E-17 1 -> -1.1102230246251568E-16 -5.5511151231257839E-17 1
